Commit message: correction of the faulty collision origin parameter in the URDF files of the rv_frl4_d...

File: src/mitsubishi_ros2_description/urdf/rv_4frl_d/rv_4frl_d.urdf.xacro (robot description, xacro)
@@ -139,5 +139,5 @@
       </visual>
       <collision>
-        <origin xyz="-0.0498 0 -0.525" rpy="1.57079633 0 0" />
+        <origin xyz="0 0 ${-0.350-0.310-0.050}" rpy="${pi/2} 0 0" />
         <geometry>
           <mesh filename="file://$(find mitsubishi_ros2_description)/meshes/rv_4frl_d/RV-4FRL_05_NO2ARM.stl" scale="0.001 0.001 0.001"/>
@@ -168,5 +168,5 @@
       </visual>
       <collision>
-        <origin xyz="-0.0498 -0.795 0" rpy="0 0 0" />
+        <origin xyz="0.335 ${-0.350-0.310-0.050} 0.0 " rpy="0 0 0" />
         <geometry>
           <mesh filename="file://$(find mitsubishi_ros2_description)/meshes/rv_4frl_d/RV-4FRL_06_WRIST.stl" scale="0.001 0.001 0.001"/>
@@ -196,5 +196,5 @@
       </visual>
       <collision>
-        <origin xyz="-0.05 -0.05 -0.795" rpy="1.5 0 0" />
+        <origin xyz="${0.335+0.08} ${-0.350-0.310-0.050} 0" rpy="0 0 0" />
         <geometry>
           <mesh filename="file://$(find mitsubishi_ros2_description)/meshes/rv_4frl_d/RV-4FRL_07_HAND_FLANGE.stl" scale="0.001 0.001 0.001"/>
